Commit message: urdf

File: urdf/aidin_m1 (backup).urdf (robot description, URDF)
Before this commit: robot aidin_m1, 14 links, 13 joints
Links:
- link LB_hip: mass 1.80 -> 0.600; geometry collision box size=0.250 0.050 0.050; visual box size=0.250 0.050 0.050
- link LB_knee: mass 1.80 -> 0.600; geometry collision box size=0.250 0.050 0.050; visual box size=0.250 0.050 0.050
- link LB_scap: mass 1.80 -> 6; geometry collision cylinder length=0.0760 radius=0.0730; visual box size=0.140 0.140 0.230
- link LF_hip: mass 1.80 -> 0.600; geometry collision box size=0.250 0.050 0.050; visual box size=0.250 0.050 0.050
- link LF_knee: mass 1.80 -> 0.600; geometry collision box size=0.250 0.050 0.050; visual box size=0.250 0.050 0.050
- link LF_scap: mass 1.80 -> 6; geometry collision cylinder length=0.0760 radius=0.0730; visual box size=0.140 0.140 0.230
- link RB_hip: mass 1.80 -> 0.600; geometry collision box size=0.250 0.050 0.050; visual box size=0.250 0.050 0.050
- link RB_knee: mass 1.80 -> 0.600; geometry collision box size=0.250 0.050 0.050; visual box size=0.250 0.050 0.050
- link RB_scap: mass 1.80 -> 6; geometry collision cylinder length=0.0760 radius=0.0730; visual box size=0.140 0.140 0.230
Joints:
- joint LBJ_hip: limit (none) -> lower=-3.14 upper=3.14 effort=200.0 velocity=9; origin xyz=0 0 0.122 rpy=1.5708 0 0 -> xyz=0.095 0 0 rpy=-1.559    1.57079  1.58259; type continuous -> revolute
- joint LBJ_knee: limit (none) -> lower=-1.308996939 upper=1.0471975512 effort=200.0 velocity=9; origin xyz=0 0 0.091 rpy=0 0 0 -> xyz=0.250 0 0 rpy=0 0 1.57079; type continuous -> revolute
- joint LBJ_scap: limit (none) -> lower=-0.00001 upper=1.5709 effort=200.0 velocity=9; origin xyz=-0.138 0.08750 0 rpy=0 1.5708 3.14159 -> xyz=-0.282 0.1150 0 rpy=1.57079 0 1.57079; type continuous -> revolute
- joint LFJ_hip: limit (none) -> lower=-3.14 upper=3.14 effort=200.0 velocity=9; origin xyz=0 0 0.122 rpy=-1.5708 0 0 -> xyz=0.095 0 0 rpy=-1.57079 1.57079 1.57079; type continuous -> revolute
- joint LFJ_knee: limit (none) -> lower=-1.308996939 upper=1.0471975512 effort=200.0 velocity=9; origin xyz=0 0 0.091 rpy=0 0 0 -> xyz=0.250 0 0 rpy=0 0 1.57079; type continuous -> revolute
- joint LFJ_scap: limit (none) -> lower=-0.00001 upper=3.14 effort=200.0 velocity=9; origin xyz=0.138 0.08750 0 rpy=0 1.5708 0 -> xyz=0.282 0.115 0 rpy=1.57079 0 1.57079; type continuous -> revolute
- joint RBJ_hip: limit (none) -> lower=-3.14 upper=3.14 effort=200.0 velocity=9; origin xyz=0 0 0.122 rpy=-1.5708 0 0 -> xyz=0.095 0 0 rpy=-1.58259 1.57079 -1.58259; type continuous -> revolute
- joint RBJ_knee: limit (none) -> lower=-1.308996939 upper=1.0471975512 effort=200.0 velocity=9; origin xyz=0 0 0.091 rpy=0 0 0 -> xyz=0.250 0 0 rpy=0 0 1.57079; type continuous -> revolute
- joint RBJ_scap: limit (none) -> lower=-1.5709 upper=0.00001 effort=200.0 velocity=9; origin xyz=-0.138 -0.08750 0 rpy=0 1.5708 3.14159 -> xyz=-0.282 -0.1150   0 rpy=-1.57079 0 -1.57079; type continuous -> revolute
- joint RFJ_hip: limit lower=-3.14 upper=0.78540 effort=200.0 velocity=9 -> lower=-3.14 upper=3.14 effort=200.0 velocity=9
- joint RFJ_knee: origin xyz=0.275 0   0 rpy=0      0      1.57079 -> xyz=0.250 0   0 rpy=0      0      1.57079
- joint RFJ_scap: limit lower=-3.14 upper=0.000001 effort=50.0 velocity=3 -> lower=-3.14 upper=0.00001 effort=200.0 velocity=9; origin xyz=0.282 -0.115 0 rpy=-1.57079 0 -1.57079 -> xyz=0.282 -0.1150 0 rpy=-1.57079 0 -1.57079

File: urdf/aidin_m1.urdf (robot description, URDF)
Before this commit: robot aidin_m1, 14 links, 13 joints
Links:
- link RB_hip: mass 1.80 -> 0.600; geometry collision box size=0.250 0.050 0.050; visual box size=0.250 0.050 0.050
- link RB_knee: mass 1.80 -> 0.600; geometry collision box size=0.250 0.050 0.050; visual box size=0.250 0.050 0.050
- link RB_scap: mass 1.80 -> 6; geometry collision cylinder length=0.0760 radius=0.0730; visual box size=0.140 0.140 0.230
Joints:
- joint LBJ_scap: limit lower=-0.00001 upper=0.6108652382 effort=200.0 velocity=9 -> lower=-0.00001 upper=1.5709 effort=200.0 velocity=9
- joint LFJ_knee: origin xyz=0.250 0   0 rpy=0 0 1.57079 -> xyz=0.250 0 0 rpy=0 0 1.57079
- joint RBJ_hip: limit (none) -> lower=-3.14 upper=3.14 effort=200.0 velocity=9; origin xyz=0 0 0.122 rpy=-1.5708 0 0 -> xyz=0.095 0 0 rpy=-1.58259 1.57079 -1.58259; type continuous -> revolute
- joint RBJ_knee: limit (none) -> lower=-1.308996939 upper=1.0471975512 effort=200.0 velocity=9; origin xyz=0 0 0.091 rpy=0 0 0 -> xyz=0.250 0 0 rpy=0 0 1.57079; type continuous -> revolute
- joint RBJ_scap: limit (none) -> lower=-1.5709 upper=0.00001 effort=200.0 velocity=9; origin xyz=-0.138 -0.08750 0 rpy=0 1.5708 3.14159 -> xyz=-0.282 -0.1150   0 rpy=-1.57079 0 -1.57079; type continuous -> revolute
- joint RFJ_hip: limit lower=-3.14 upper=0.78540 effort=200.0 velocity=9 -> lower=-3.14 upper=3.14 effort=200.0 velocity=9
- joint RFJ_scap: limit lower=-3.14 upper=0.000001 effort=50.0 velocity=3 -> lower=-3.14 upper=0.00001 effort=200.0 velocity=9

Commit message: backup

File: urdf/aidin_m1 (backup).urdf (robot description, URDF)
Before this commit: robot aidin_m1, 14 links, 13 joints
Joints:
- joint LFJ_scap: limit lower=-0.00001 upper=3.14 effort=200.0 velocity=9 -> lower=-0.00001 upper=1.5709 effort=200.0 velocity=9
- joint RFJ_scap: limit lower=-3.14 upper=0.00001 effort=200.0 velocity=9 -> lower=-1.5709 upper=0.00001 effort=200.0 velocity=9
