Commit message: 우선 inertial는 이전 버전으로 백섭

File: urdf/aidin_m1_backup.urdf (robot description, URDF)
Before this commit: robot aidin_m1, 18 links, 17 joints
Links:
- link LB_hip: mass 0.600 -> 0.644
- link LB_knee: mass 0.600 -> 0.343
- link LF_hip: mass 0.600 -> 0.644
- link LF_knee: mass 0.600 -> 0.343s
- link RB_hip: mass 0.600 -> 0.615
- link RB_knee: mass 0.600 -> 0.343
- link RF_hip: mass 0.600 -> 0.615
- link RF_knee: mass 0.600 -> 0.343
