Commit message: test

File: urdf/aidin_m1.urdf (robot description, URDF)
Before this commit: robot aidin_m1, 14 links, 13 joints
Joints:
- joint RFJ_scap: origin xyz=0.282 -0.08750 0 rpy=-1.57079 0 -1.57079 -> xyz=0.282 -0.115 0 rpy=-1.57079 0 -1.57079

Commit message: LF

File: urdf/aidin_m1.urdf (robot description, URDF)
Before this commit: robot aidin_m1, 14 links, 13 joints
Links:
- link LF_hip: mass 1.80 -> 0.600; geometry collision box size=0.250 0.050 0.050; visual box size=0.250 0.050 0.050
- link LF_knee: mass 1.80 -> 0.600; geometry collision box size=0.250 0.050 0.050; visual box size=0.250 0.050 0.050
- link LF_scap: mass 1.80 -> 6; geometry collision cylinder length=0.0760 radius=0.0730; visual box size=0.140 0.140 0.230
Joints:
- joint LFJ_hip: limit (none) -> lower=-3.14 upper=3.14 effort=200.0 velocity=9; origin xyz=0 0 0.122 rpy=-1.5708 0 0 -> xyz=0.095 0 0 rpy=-1.57079 1.57079 1.57079; type continuous -> revolute
- joint LFJ_knee: limit (none) -> lower=-1.308996939 upper=1.0471975512 effort=200.0 velocity=9; origin xyz=0 0 0.091 rpy=0 0 0 -> xyz=0.275 0   0 rpy=0 0 1.57079; type continuous -> revolute
- joint LFJ_scap: limit (none) -> lower=-0.00001 upper=3.14 effort=200.0 velocity=9; origin xyz=0.138 0.08750 0 rpy=0 1.5708 0 -> xyz=0.282 0.115 0 rpy=1.57079 0 1.57079; type continuous -> revolute
- joint RFJ_scap: origin xyz=0.282 -0.115 0 rpy=-1.57079 0 -1.57079 -> xyz=0.282 -0.1150 0 rpy=-1.57079 0 -1.57079

Commit message: LB

File: urdf/aidin_m1.urdf (robot description, URDF)
Before this commit: robot aidin_m1, 14 links, 13 joints
Links:
- link LB_hip: mass 1.80 -> 0.600; geometry collision box size=0.250 0.050 0.050; visual box size=0.250 0.050 0.050
- link LB_knee: mass 1.80 -> 0.600; geometry collision box size=0.250 0.050 0.050; visual box size=0.250 0.050 0.050
- link LB_scap: mass 1.80 -> 6; geometry collision cylinder length=0.0760 radius=0.0730; visual box size=0.140 0.140 0.230
Joints:
- joint LBJ_hip: limit (none) -> lower=-3.14 upper=3.14 effort=200.0 velocity=9; origin xyz=0 0 0.122 rpy=1.5708 0 0 -> xyz=0.095 0 0 rpy=-1.559    1.57079  1.58259; type continuous -> revolute
- joint LBJ_knee: limit (none) -> lower=-1.308996939 upper=1.0471975512 effort=200.0 velocity=9; origin xyz=0 0 0.091 rpy=0 0 0 -> xyz=0.250 0 0 rpy=0 0 1.57079; type continuous -> revolute
- joint LBJ_scap: limit (none) -> lower=-0.00001 upper=0.6108652382 effort=200.0 velocity=9; origin xyz=-0.138 0.08750 0 rpy=0 1.5708 3.14159 -> xyz=-0.282 0.1150 0 rpy=1.57079 0 1.57079; type continuous -> revolute
- joint LFJ_knee: origin xyz=0.275 0   0 rpy=0 0 1.57079 -> xyz=0.250 0   0 rpy=0 0 1.57079
- joint RFJ_knee: origin xyz=0.275 0   0 rpy=0      0      1.57079 -> xyz=0.250 0   0 rpy=0      0      1.57079

Commit message: edit hip joint

File: urdf/aidin_m1.urdf (robot description, URDF)
Before this commit: robot aidin_m1, 14 links, 13 joints
Joints:
- joint LBJ_scap: limit lower=-0.00001 upper=1.5709 effort=200.0 velocity=9 -> lower=-0.7854 upper=0.00001 effort=200.0 velocity=9
- joint LFJ_scap: limit lower=-0.00001 upper=1.5709 effort=200.0 velocity=9 -> lower=-0.7854 upper=0.00001 effort=200.0 velocity=9
- joint RBJ_scap: limit lower=-1.5709 upper=0.00001 effort=200.0 velocity=9 -> lower=-0.00001 upper=0.7854 effort=200.0 velocity=9
- joint RFJ_scap: limit lower=-1.5709 upper=0.00001 effort=200.0 velocity=9 -> lower=-0.00001 upper=0.7854 effort=200.0 velocity=9

Commit message: edit collision

File: urdf/aidin_m1.urdf (robot description, URDF)
Before this commit: robot aidin_m1, 14 links, 13 joints
Links:
- link LB_scap: geometry collision box size=0.140 0.140 0.230; visual box size=0.140 0.140 0.230
- link LF_scap: geometry collision box size=0.140 0.140 0.230; visual box size=0.140 0.140 0.230
- link RB_scap: geometry collision box size=0.140 0.140 0.230; visual box size=0.140 0.140 0.230
- link RF_scap: geometry collision box size=0.140 0.140 0.230; visual box size=0.140 0.140 0.230

Commit message: edit collision of knee link

File: urdf/aidin_m1.urdf (robot description, URDF)
Before this commit: robot aidin_m1, 14 links, 13 joints
Links:
- link LB_knee: geometry collision box size=0.230 0.050 0.050; visual box size=0.250 0.050 0.050
- link LF_knee: geometry collision box size=0.230 0.050 0.050; visual box size=0.250 0.050 0.050
- link RB_knee: geometry collision box size=0.230 0.050 0.050; visual box size=0.250 0.050 0.050
- link RF_knee: geometry collision box size=0.230 0.050 0.050; visual box size=0.250 0.050 0.050

Commit message: edit limit of revolute joint

File: urdf/aidin_m1.urdf (robot description, URDF)
Before this commit: robot aidin_m1, 14 links, 13 joints
Joints:
- joint LBJ_scap: limit lower=-0.7854 upper=0.00001 effort=200.0 velocity=9 -> lower=-0.7854 upper=0 effort=200.0 velocity=9
- joint LFJ_scap: limit lower=-0.7854 upper=0.00001 effort=200.0 velocity=9 -> lower=-0.7854 upper=0 effort=200.0 velocity=9
- joint RBJ_scap: limit lower=-0.00001 upper=0.7854 effort=200.0 velocity=9 -> lower=0 upper=0.7854 effort=200.0 velocity=9
- joint RFJ_scap: limit lower=-0.00001 upper=0.7854 effort=200.0 velocity=9 -> lower=0 upper=0.7854 effort=200.0 velocity=9

Commit message: add foot link&joint

File: urdf/aidin_m1.urdf (robot description, URDF)
Before this commit: robot aidin_m1, 14 links, 13 joints
Links:
- added link LB_foot, mass 0.01; collision sphere radius=0.025; visual sphere radius=0.0250
- added link LF_foot, mass 0.01; collision sphere radius=0.025; visual sphere radius=0.0250
- added link RB_foot, mass 0.01; collision sphere radius=0.025; visual sphere radius=0.0250
- added link RF_foot, mass 0.01; collision sphere radius=0.025; visual sphere radius=0.0250
Joints:
- added joint LBJ_foot: type fixed, parent LB_knee, child LB_foot, origin xyz=0.25 0 0 rpy=0 0 0, axis 0 0 1
- added joint LFJ_foot: type fixed, parent LF_knee, child LF_foot, origin xyz=0.25 0 0 rpy=0 0 0, axis 0 0 1
- added joint RBJ_foot: type fixed, parent RB_knee, child RB_foot, origin xyz=0.25 0 0 rpy=0 0 0, axis 0 0 1
- added joint RFJ_foot: type fixed, parent RF_knee, child RF_foot, origin xyz=0.25 0 0 rpy=0 0 0, axis 0 0 1
- joint odom_joint: origin xyz=0 0 0.440 rpy=0 0 0 -> xyz=0 0 0.500 rpy=0 0 0

Commit message: edit REDAME

File: urdf/aidin_m1.urdf (robot description, URDF)
Before this commit: robot aidin_m1, 18 links, 17 joints
Joints:
- joint odom_joint: origin xyz=0 0 0.500 rpy=0 0 0 -> xyz=0 0 0.550 rpy=0 0 0

Commit message: edit RFJ joint from revolute to continuous

File: urdf/aidin_m1.urdf (robot description, URDF)
Before this commit: robot aidin_m1, 18 links, 17 joints
Joints:
- joint RFJ_hip: limit lower=-3.14 upper=3.14 effort=200.0 velocity=9 -> (none); type revolute -> continuous
- joint RFJ_knee: axis 0 0 1 -> (none); limit lower=-1.308996939 upper=1.0471975512 effort=200.0 velocity=9 -> (none); origin xyz=0.250 0   0 rpy=0      0      1.57079 -> xyz=0.250 0 0 rpy=0 0 1.57079; type revolute -> continuous

Commit message: edit Inverse Kinematics Calculation (2)

File: urdf/aidin_m1.urdf (robot description, URDF)
Before this commit: robot aidin_m1, 18 links, 17 joints
Joints:
- joint RBJ_knee: limit lower=-1.308996939 upper=1.0471975512 effort=200.0 velocity=9 -> lower=-3.14 upper=3.14 effort=200.0 velocity=9

Commit message: 중간 저장

File: urdf/aidin_m1.urdf (robot description, URDF)
Before this commit: robot aidin_m1, 18 links, 17 joints
Joints:
- joint LBJ_hip: limit lower=-3.14 upper=3.14 effort=200.0 velocity=9 -> (none); origin xyz=0.095 0 0 rpy=-1.559    1.57079  1.58259 -> xyz=0.095 0 0 rpy=-1.559 1.57079 1.58259; type revolute -> continuous
- joint LBJ_knee: limit lower=-1.308996939 upper=1.0471975512 effort=200.0 velocity=9 -> (none); type revolute -> continuous
- joint LFJ_hip: limit lower=-3.14 upper=3.14 effort=200.0 velocity=9 -> (none); type revolute -> continuous
- joint LFJ_knee: limit lower=-1.308996939 upper=1.0471975512 effort=200.0 velocity=9 -> (none); type revolute -> continuous
- joint RBJ_hip: limit lower=-3.14 upper=3.14 effort=200.0 velocity=9 -> (none); type revolute -> cotinuous
- joint RBJ_knee: limit lower=-3.14 upper=3.14 effort=200.0 velocity=9 -> (none); type revolute -> continuous
- joint RFJ_knee: axis (none) -> 0 0 1

Commit message: urdf 수정 전 백업

File: urdf/aidin_m1.urdf (robot description, URDF)
Before this commit: robot aidin_m1, 18 links, 17 joints
Joints:
- joint LFJ_hip: limit (none) -> lower=-3.14 upper=3.14 effort=200.0 velocity=9; type continuous -> revolute
- joint LFJ_knee: limit (none) -> lower=-1.308996939 upper=1.0471975512 effort=200.0 velocity=9; type continuous -> revolute
- joint RBJ_hip: limit (none) -> lower=-3.14 upper=3.14 effort=200.0 velocity=9; type cotinuous -> revolute
- joint RBJ_knee: limit (none) -> lower=-3.14 upper=3.14 effort=200.0 velocity=9; type continuous -> revolute

Commit message: urdf 수정 완료 (revolute to continuous)

File: urdf/aidin_m1.urdf (robot description, URDF)
Before this commit: robot aidin_m1, 18 links, 17 joints
Joints:
- joint LFJ_hip: limit lower=-3.14 upper=3.14 effort=200.0 velocity=9 -> (none); type revolute -> continuous
- joint LFJ_knee: limit lower=-1.308996939 upper=1.0471975512 effort=200.0 velocity=9 -> (none); type revolute -> continuous
- joint RBJ_hip: limit lower=-3.14 upper=3.14 effort=200.0 velocity=9 -> (none); type revolute -> continuous
- joint RBJ_knee: limit lower=-3.14 upper=3.14 effort=200.0 velocity=9 -> (none); type revolute -> continuous

Commit message: 수정 완료

File: urdf/aidin_m1.urdf (robot description, URDF)
Before this commit: robot aidin_m1, 18 links, 17 joints
Joints:
- joint LBJ_hip: limit (none) -> lower=-3.14 upper=3.14 effort=200.0 velocity=9; type continuous -> revolute
- joint LBJ_knee: limit (none) -> lower=-1.308996939 upper=1.0471975512 effort=200.0 velocity=9; type continuous -> revolute
- joint LFJ_hip: limit (none) -> lower=-3.14 upper=3.14 effort=200.0 velocity=9; type continuous -> revolute
- joint LFJ_knee: limit (none) -> lower=-1.308996939 upper=1.0471975512 effort=200.0 velocity=9; type continuous -> revolute
- joint RBJ_hip: limit (none) -> lower=-3.14 upper=3.14 effort=200.0 velocity=9; type continuous -> revolute
- joint RBJ_knee: limit (none) -> lower=-3.14 upper=3.14 effort=200.0 velocity=9; type continuous -> revolute
- joint RFJ_hip: limit (none) -> lower=-3.14 upper=3.14 effort=200.0 velocity=9; type continuous -> revolute
- joint RFJ_knee: limit (none) -> lower=-1.308996939 upper=1.0471975512 effort=200.0 velocity=9; type continuous -> revolute

Commit message: msg->data 입력 list로 변경 (=code 단순화)

File: urdf/aidin_m1.urdf (robot description, URDF)
Before this commit: robot aidin_m1, 18 links, 17 joints
Joints:
- joint LBJ_knee: limit lower=-1.308996939 upper=1.0471975512 effort=200.0 velocity=9 -> lower=-3.14 upper=3.14 effort=200.0 velocity=9
- joint LBJ_scap: limit lower=-0.7854 upper=0 effort=200.0 velocity=9 -> lower=-1.57089 upper=1.57089 effort=200.0 velocity=9
- joint LFJ_knee: limit lower=-1.308996939 upper=1.0471975512 effort=200.0 velocity=9 -> lower=-3.14 upper=3.14 effort=200.0 velocity=9
- joint LFJ_scap: limit lower=-0.7854 upper=0 effort=200.0 velocity=9 -> lower=-1.57089 upper=1.57089 effort=200.0 velocity=9
- joint RBJ_scap: limit lower=0 upper=0.7854 effort=200.0 velocity=9 -> lower=-1.57089 upper=1.57089 effort=200.0 velocity=9
- joint RFJ_knee: limit lower=-1.308996939 upper=1.0471975512 effort=200.0 velocity=9 -> lower=-3.14 upper=3.14 effort=200.0 velocity=9
- joint RFJ_scap: limit lower=0 upper=0.7854 effort=200.0 velocity=9 -> lower=-1.57089 upper=1.57089 effort=200.0 velocity=9

Commit message: FeedforwardController build 성공

File: urdf/aidin_m1.urdf (robot description, URDF)
Before this commit: robot aidin_m1, 18 links, 17 joints
Links:
- link RF_hip: mass 0.600 -> 1.000
- link RF_knee: mass 0.600 -> 1.000

Commit message: urdf visual update 완료 (1)

File: urdf/aidin_m1.urdf (robot description, URDF)
Before this commit: robot aidin_m1, 18 links, 17 joints
Links:
- link LB_hip: geometry collision box size=0.250 0.050 0.050; visual mesh filename=/home/eunseop/dev_ws/src/aidin_m1/meshes/LF_hip_vis.stl scale=0.001 0.001 0.001
- link LB_knee: geometry collision box size=0.230 0.050 0.050; visual mesh filename=/home/eunseop/dev_ws/src/aidin_m1/meshes/LF_knee_vis.stl scale=0.001 0.001 0.001
- link LB_scap: geometry collision box size=0.140 0.140 0.230; visual mesh filename=/home/eunseop/dev_ws/src/aidin_m1/meshes/LB_scap_vis.stl scale=0.001 0.001 0.001
- link LF_hip: geometry collision box size=0.250 0.050 0.050; visual mesh filename=/home/eunseop/dev_ws/src/aidin_m1/meshes/LF_hip_vis.stl scale=0.001 0.001 0.001
- link LF_knee: geometry collision box size=0.230 0.050 0.050; visual mesh filename=/home/eunseop/dev_ws/src/aidin_m1/meshes/LF_knee_vis.stl scale=0.001 0.001 0.001
- link LF_scap: geometry collision box size=0.140 0.140 0.230; visual mesh filename=/home/eunseop/dev_ws/src/aidin_m1/meshes/LF_scap_vis.stl scale=0.001 0.001 0.001
- link RB_hip: geometry collision box size=0.250 0.050 0.050; visual mesh filename=/home/eunseop/dev_ws/src/aidin_m1/meshes/RF_hip_vis.stl scale=0.001 0.001 0.001
- link RB_knee: geometry collision box size=0.230 0.050 0.050; visual mesh filename=/home/eunseop/dev_ws/src/aidin_m1/meshes/LF_knee_vis.stl scale=0.001 0.001 0.001
- link RB_scap: geometry collision box size=0.140 0.140 0.230; visual mesh filename=/home/eunseop/dev_ws/src/aidin_m1/meshes/RB_scap_vis.stl scale=0.001 0.001 0.001
- link RF_hip: mass 1.000 -> 0.600; geometry collision box size=0.250 0.050 0.050; visual mesh filename=/home/eunseop/dev_ws/src/aidin_m1/meshes/RF_hip_vis.stl scale=0.001 0.001 0.001
- link RF_knee: mass 1.000 -> 0.600; geometry collision box size=0.230 0.050 0.050; visual mesh filename=/home/eunseop/dev_ws/src/aidin_m1/meshes/RF_knee_vis.stl scale=0.001 0.001 0.001
- link RF_scap: geometry collision box size=0.140 0.140 0.230; visual mesh filename=/home/eunseop/dev_ws/src/aidin_m1/meshes/RF_scap_vis.stl scale=0.001 0.001 0.001
- link body: geometry collision box size=0.200 0.370 0.216; visual mesh filename=/home/eunseop/dev_ws/src/aidin_m1/meshes/Body_vis.stl scale=0.001 0.001 0.001
Joints:
- joint LBJ_scap: origin xyz=-0.282 0.1150 0 rpy=1.57079 0 1.57079 -> xyz=-0.255 0.120 0 rpy=1.57079 0 1.57079
- joint LFJ_scap: origin xyz=0.282 0.115 0 rpy=1.57079 0 1.57079 -> xyz=0.255 0.120 0 rpy=1.57079 0 1.57079
- joint RBJ_scap: origin xyz=-0.282 -0.1150   0 rpy=-1.57079 0 -1.57079 -> xyz=-0.255 -0.120   0 rpy=-1.57079 0 -1.57079
- joint RFJ_scap: origin xyz=0.282 -0.1150 0 rpy=-1.57079 0 -1.57079 -> xyz=0.255 -0.120 0 rpy=-1.57079 0 -1.57079

Commit message: 발 방향 수정

File: urdf/aidin_m1.urdf (robot description, URDF)
Before this commit: robot aidin_m1, 18 links, 17 joints
Links:
- link LB_foot: mass 0.01 -> 0; geometry collision sphere radius=0.025; visual mesh filename=/home/eunseop/dev_ws/src/aidin_m1/meshes/feet.stl scale=0.001 0.001 0.001
- link LF_foot: mass 0.01 -> 0; geometry collision sphere radius=0.025; visual mesh filename=/home/eunseop/dev_ws/src/aidin_m1/meshes/feet.stl scale=0.001 0.001 0.001
- link RB_foot: mass 0.01 -> 0; geometry collision sphere radius=0.025; visual mesh filename=/home/eunseop/dev_ws/src/aidin_m1/meshes/feet.stl scale=0.001 0.001 0.001
- link RF_foot: mass 0.01 -> 0; geometry collision sphere radius=0.025; visual mesh filename=/home/eunseop/dev_ws/src/aidin_m1/meshes/feet.stl scale=0.001 0.001 0.001
Joints:
- joint LBJ_foot: origin xyz=0.25 0 0 rpy=0 0 0 -> xyz=0.250 -0.010 0.002 rpy=-1.57089 0 -1.57089
- joint LFJ_foot: origin xyz=0.25 0 0 rpy=0 0 0 -> xyz=0.250 -0.010 0.002 rpy=-1.57089 0 -1.57089
- joint RBJ_foot: origin xyz=0.25 0 0 rpy=0 0 0 -> xyz=0.250 -0.010 0.002 rpy=-1.57089 0 -1.57089
- joint RFJ_foot: origin xyz=0.25 0 0 rpy=0 0 0 -> xyz=0.250 -0.010 0.002 rpy=-1.57089 0 -1.57089

Commit message: mass & inertial update (from Inventor)

File: urdf/aidin_m1.urdf (robot description, URDF)
Before this commit: robot aidin_m1, 18 links, 17 joints
Links:
- link LB_hip: mass 0.600 -> 0.644
- link LB_knee: mass 0.600 -> 0.343
- link LB_scap: mass 6 -> 2.739
- link LF_hip: mass 0.600 -> 0.644
- link LF_knee: mass 0.600 -> 0.343s
- link LF_scap: mass 6 -> 2.694
- link RB_hip: mass 0.600 -> 0.615
- link RB_knee: mass 0.600 -> 0.343
- link RB_scap: mass 6 -> 2.739
- link RF_hip: mass 0.600 -> 0.615
- link RF_knee: mass 0.600 -> 0.343
- link RF_scap: mass 6 -> 2.739

Commit message: inertial 값 오류 안 나오는 값으로 변경 -> Feedforward 이 값으로 진행

File: urdf/aidin_m1.urdf (robot description, URDF)
Before this commit: robot aidin_m1, 18 links, 17 joints
Links:
- link LB_hip: mass 0.600 -> 0.644
- link LB_knee: mass 0.600 -> 0.343
- link LF_hip: mass 0.600 -> 0.644
- link LF_knee: mass 0.600 -> 0.343
- link RB_hip: mass 0.600 -> 0.644
- link RB_knee: mass 0.600 -> 0.343
- link RF_foot: mass 0 -> 0.01
- link RF_hip: mass 0.600 -> 0.644; geometry collision box size=0.250 0.030 0.030; visual mesh filename=/home/eunseop/dev_ws/src/aidin_m1/meshes/RF_hip_vis.stl scale=0.001 0.001 0.001
- link RF_knee: mass 0.600 -> 0.343; geometry collision box size=0.230 0.030 0.030; visual mesh filename=/home/eunseop/dev_ws/src/aidin_m1/meshes/RF_knee_vis.stl scale=0.001 0.001 0.001

File: urdf/aidin_m1_backup.urdf (robot description, URDF)
Before this commit: robot aidin_m1, 18 links, 17 joints
Links:
- link LF_knee: mass 0.343s -> 0.343

Commit message: hip&knee link collision size 변경

File: urdf/aidin_m1.urdf (robot description, URDF)
Before this commit: robot aidin_m1, 18 links, 17 joints
Links:
- link LB_hip: geometry collision box size=0.250 0.030 0.030; visual mesh filename=/home/eunseop/dev_ws/src/aidin_m1/meshes/LF_hip_vis.stl scale=0.001 0.001 0.001
- link LB_knee: geometry collision box size=0.230 0.030 0.030; visual mesh filename=/home/eunseop/dev_ws/src/aidin_m1/meshes/LF_knee_vis.stl scale=0.001 0.001 0.001
- link LF_hip: geometry collision box size=0.250 0.030 0.030; visual mesh filename=/home/eunseop/dev_ws/src/aidin_m1/meshes/LF_hip_vis.stl scale=0.001 0.001 0.001
- link LF_knee: geometry collision box size=0.230 0.030 0.030; visual mesh filename=/home/eunseop/dev_ws/src/aidin_m1/meshes/LF_knee_vis.stl scale=0.001 0.001 0.001
- link RB_hip: geometry collision box size=0.250 0.030 0.030; visual mesh filename=/home/eunseop/dev_ws/src/aidin_m1/meshes/RF_hip_vis.stl scale=0.001 0.001 0.001
- link RB_knee: geometry collision box size=0.230 0.030 0.030; visual mesh filename=/home/eunseop/dev_ws/src/aidin_m1/meshes/LF_knee_vis.stl scale=0.001 0.001 0.001

Commit message: Feedforwardtorquecontrol3D 수정->테스트 전 백업

File: urdf/aidin_m1.urdf (robot description, URDF)
Before this commit: robot aidin_m1, 18 links, 17 joints
Links:
- link RF_foot: mass 0.01 -> 0

Commit message: RF만 강체(직육면체)로 변환

File: urdf/aidin_m1.urdf (robot description, URDF)
Before this commit: robot aidin_m1, 18 links, 17 joints
Links:
- link RF_hip: mass 0.644 -> 1.688; geometry collision box size=0.250 0.030 0.030; visual mesh filename=/home/eunseop/dev_ws/src/aidin_m1/meshes/RF_hip.stl scale=0.001 0.001 0.001
- link RF_knee: mass 0.343 -> 1.688; geometry collision box size=0.230 0.030 0.030; visual mesh filename=/home/eunseop/dev_ws/src/aidin_m1/meshes/RF_knee.stl scale=0.001 0.001 0.001
- link RF_scap: mass 6 -> 12.172; geometry collision box size=0.140 0.140 0.230; visual mesh filename=/home/eunseop/dev_ws/src/aidin_m1/meshes/RF_scap.stl scale=0.001 0.001 0.001

Commit message: 무게중심 정확하게 입력 in urdf

File: urdf/aidin_m1.urdf (robot description, URDF)
Before this commit: robot aidin_m1, 18 links, 17 joints
Links:
- link RF_hip: mass 1.688 -> 0.615; geometry collision box size=0.250 0.030 0.030; visual mesh filename=/home/eunseop/dev_ws/src/aidin_m1/meshes/RF_hip_vis.stl scale=0.001 0.001 0.001
- link RF_knee: mass 1.688 -> 0.343; geometry collision box size=0.230 0.030 0.030; visual mesh filename=/home/eunseop/dev_ws/src/aidin_m1/meshes/RF_knee_vis.stl scale=0.001 0.001 0.001
- link RF_scap: mass 12.172 -> 2.739; geometry collision box size=0.140 0.140 0.230; visual mesh filename=/home/eunseop/dev_ws/src/aidin_m1/meshes/RF_scap_vis.stl scale=0.001 0.001 0.001

Commit message: feedforward LB link에도 적용 (just 대칭)

File: urdf/aidin_m1.urdf (robot description, URDF)
Before this commit: robot aidin_m1, 18 links, 17 joints
Links:
- link LB_hip: mass 0.644 -> 0.615
- link LB_scap: mass 6 -> 2.739

Commit message: feedforward 다리 4개에 모두 적용 (just 대칭)

File: urdf/aidin_m1.urdf (robot description, URDF)
Before this commit: robot aidin_m1, 18 links, 17 joints
Links:
- link LF_hip: mass 0.644 -> 0.615
- link LF_scap: mass 6 -> 2.739
- link RB_hip: mass 0.644 -> 0.615
- link RB_scap: mass 6 -> 2.739

Commit message: Body 고정 풀고 평지 보행 성공 (경로 제어는 안 됨)

File: urdf/aidin_m1.urdf (robot description, URDF)
Before this commit: robot aidin_m1, 18 links, 17 joints
Links:
- added link dummy_base_1, mass 0.01
- added link dummy_base_2, mass 0.01
Joints:
- removed joint odom_joint
- added joint x_joint_move: type prismatic, parent world, child dummy_base_1, origin xyz=0 0 0 rpy=0 0 0, axis 1 0 0, limit lower=-1000 upper=1000 effort=200000 velocity=10000
- added joint y_joint_move: type prismatic, parent dummy_base_1, child dummy_base_2, origin xyz=0 0 0 rpy=0 0 0, axis 0 1 0, limit lower=-1000 upper=1000 effort=200000 velocity=10000
- added joint z_joint_revolute: type continuous, parent dummy_base_2, child body, origin xyz=0 0 0.450 rpy=0 0 0, axis 0 0 1, limit effort=200 velocity=10

File: urdf/aidin_m1.xacro (robot description, xacro)
@@ -1,4 +1,4 @@
 <?xml version="1.0"?>
-<robot name="aidin_m1">
+<robot name="aidin_m1" xmlns:xacro="http://www.ros.org/wiki/xacro">
   <material name="black">
     <color rgba="0.0 0.0 0.0 1.0"/>
@@ -65,5 +65,6 @@
       <geometry>
         <!-- <box size="0.200 0.370 0.216"/> -->
-        <mesh filename="/home/eunseop/dev_ws/src/aidin_m1/meshes/Body_vis.stl" scale="0.001 0.001 0.001"/>
+        <!-- <mesh filename="/home/eunseop/dev_ws/src/aidin_m1/meshes/Body_vis.stl" scale="0.001 0.001 0.001"/> -->
+        <mesh filename="package://aidin_m1/meshes/Body_vis.stl"/>
       </geometry>
       <material name="silver"/>
@@ -78,8 +79,6 @@
       <mass value="2.739"/>
       <origin xyz="-0.002 0 -0.031" rpy="0 0 0"/>
-      <!-- <inertia ixx="0" ixy="0" ixz="0" iyy="0" iyz="0" izz="0"/> -->
       <!-- <inertia ixx="0.73716790" ixy="0.130721360" ixz="0" iyy="0.431162858" iyz="0" izz="0.477083568"/> -->
       <inertia ixx="0.018386717" ixy="-0.000009042" ixz="-0.000004977" iyy="0.020489644" iyz="-0.000009312" izz="0.008551259"/>
-      <!-- <inertia ixx="0.73716790" ixy="0.130721360" ixz="0" iyy="0.431162858" iyz="0" izz="0.477083568"/> -->
     </inertial>
     <collision>

Commit message: 정지 명령어 추가 & 직선 보행 성공

File: urdf/aidin_m1.urdf (robot description, URDF)
Before this commit: robot aidin_m1, 20 links, 19 joints
Joints:
- joint z_joint_revolute: origin xyz=0 0 0.450 rpy=0 0 0 -> xyz=0 0 0.500 rpy=0 0 0
