Commit message: urdf damping 1.5 -> 3

File: urdf/aidin_m1.urdf (robot description, URDF)
Before this commit: robot aidin_m1, 20 links, 19 joints
Joints:
- joint z_joint_revolute: origin xyz=0 0 0.500 rpy=0 0 0 -> xyz=0 0 0.480 rpy=0 0 0

File: urdf/aidin_m1.xacro (robot description, xacro)
@@ -66,5 +66,5 @@
         <!-- <box size="0.200 0.370 0.216"/> -->
         <!-- <mesh filename="/home/eunseop/dev_ws/src/aidin_m1/meshes/Body_vis.stl" scale="0.001 0.001 0.001"/> -->
-        <mesh filename="package://aidin_m1/meshes/Body_vis.stl"/>
+        <!-- <mesh filename="package://aidin_m1/meshes/Body_vis.stl"/> -->
       </geometry>
       <material name="silver"/>

Commit message: 잘 걷고 잘 멈춤

File: urdf/aidin_m1.urdf (robot description, URDF)
Before this commit: robot aidin_m1, 20 links, 19 joints
Joints:
- joint z_joint_revolute: origin xyz=0 0 0.480 rpy=0 0 0 -> xyz=0 0 0.450 rpy=0 0 0

Commit message: urdf 수정 전 백업

File: urdf/aidin_m1.urdf (robot description, URDF)
Before this commit: robot aidin_m1, 20 links, 19 joints
Links:
- removed link dummy_base_1
- removed link dummy_base_2
Joints:
- removed joint x_joint_move
- removed joint y_joint_move
- joint z_joint_revolute: parent dummy_base_2 -> world

Commit message: body 고정은 풀렸는데, 잘 못걷고 넘어짐

File: urdf/aidin_m1.urdf (robot description, URDF)
Before this commit: robot aidin_m1, 18 links, 17 joints
Links:
- removed link world
- added link base; visual box size=0.001 0.001 0.001
Joints:
- removed joint z_joint_revolute
- added joint floating_base: type fixed, parent base, child body, origin xyz=0 0 0 rpy=0 0 0

Commit message: imu joint & imu link 추가

File: urdf/aidin_m1.urdf (robot description, URDF)
Before this commit: robot aidin_m1, 18 links, 17 joints
Links:
- added link imu_link, mass 0.001; collision box size=0.001 0.001 0.001; visual box size=0.001 0.001 0.001
Joints:
- added joint imu_joint: type fixed, parent body, child imu_link, origin xyz=0 0 0 rpy=0 0 0

Commit message: foot joint dont_collapse 삭제

File: urdf/aidin_m1.urdf (robot description, URDF)
Before this commit: robot aidin_m1, 19 links, 18 joints
Joints:
- joint LBJ_foot: axis 0 0 1 -> (none)
- joint LFJ_foot: axis 0 0 1 -> (none)
- joint RBJ_foot: axis 0 0 1 -> (none)
- joint RFJ_foot: axis 0 0 1 -> (none)

Commit message: aidin_m1.urdf: rod cell 추가

File: urdf/aidin_m1.urdf (robot description, URDF)
Before this commit: robot aidin_m1, 18 links, 17 joints
Links:
- added link LB_rod_cell, mass 0.001; collision cylinder length=0.002 radius=0.005; visual cylinder length=0.002 radius=0.005
- added link LF_rod_cell, mass 0.001; collision cylinder length=0.002 radius=0.005; visual cylinder length=0.002 radius=0.005
- added link RB_rod_cell, mass 0.001; collision cylinder length=0.002 radius=0.005; visual cylinder length=0.002 radius=0.005
- added link RF_rod_cell, mass 0.001; collision cylinder length=0.002 radius=0.005; visual cylinder length=0.002 radius=0.005
- added link upper_body, mass 0.0001; collision box size=0.200 0.370 0.010; visual box size=0.200 0.370 0.010
- link body: geometry collision box size=0.200 0.370 0.160; visual mesh filename=/home/eunseop/dev_ws/src/aidin_m1/meshes/Body_vis.stl scale=0.001 0.001 0.001
Joints:
- added joint LBJ_rod_cell: type fixed, parent upper_body, child LB_rod_cell, origin xyz=0 0 0 rpy=0 0 0
- added joint LFJ_rod_cell: type fixed, parent upper_body, child LF_rod_cell, origin xyz=0 0 0 rpy=0 0 0
- added joint RBJ_rod_cell: type fixed, parent upper_body, child RB_rod_cell, origin xyz=0 0 0 rpy=0 0 0
- added joint RFJ_rod_cell: type fixed, parent upper_body, child RF_rod_cell, origin xyz=0 0 0 rpy=0 0 0
- added joint upper_body_J: type fixed, parent base, child upper_body, origin xyz=0 0 0 rpy=0 0 0

Commit message: urdf에 추가할 건 다 했음

File: urdf/aidin_m1.urdf (robot description, URDF)
Before this commit: robot aidin_m1, 23 links, 22 joints
Links:
- added link object, mass 1; collision box size=0.050 0.050 0.050; visual box size=0.050 0.050 0.050
- added link upper_box, mass 0.0001; collision box size=0.190 0.120 0.010; visual box size=0.190 0.120 0.010
- link LB_rod_cell: geometry collision cylinder length=0.0050 radius=0.005; visual cylinder length=0.0050 radius=0.005
- link LF_rod_cell: geometry collision cylinder length=0.0050 radius=0.005; visual cylinder length=0.0050 radius=0.005
- link RB_rod_cell: geometry collision cylinder length=0.0050 radius=0.005; visual cylinder length=0.0050 radius=0.005
- link RF_rod_cell: geometry collision cylinder length=0.0050 radius=0.005; visual cylinder length=0.0050 radius=0.005
Joints:
- added joint object_J: type fixed, parent upper_box, child object, origin xyz=0 0 0 rpy=0 0 0
- added joint upper_box_J: type fixed, parent upper_body, child upper_box, origin xyz=0 0 0 rpy=0 0 0

Commit message: urdf 수정: fixed joint를 revolute로 바꿔서 GetLink로 인식 가능하게 함

File: urdf/aidin_m1.urdf (robot description, URDF)
Before this commit: robot aidin_m1, 25 links, 24 joints
Joints:
- joint LBJ_rod_cell: axis (none) -> 0 0 1; limit (none) -> lower=0 upper=0.0001 effort=1 velocity=0.0001; origin xyz=0 0 0 rpy=0 0 0 -> xyz=-0.075 0.050 0.0075 rpy=0 0 0; type fixed -> revolute
- joint LFJ_rod_cell: axis (none) -> 0 0 1; limit (none) -> lower=0 upper=0.0001 effort=1 velocity=0.0001; origin xyz=0 0 0 rpy=0 0 0 -> xyz=0.075 0.050 0.0075 rpy=0 0 0; type fixed -> revolute
- joint RBJ_rod_cell: axis (none) -> 0 0 1; limit (none) -> lower=0 upper=0.0001 effort=1 velocity=0.0001; origin xyz=0 0 0 rpy=0 0 0 -> xyz=-0.075 -0.050 0.0075 rpy=0 0 0; type fixed -> revolute
- joint RFJ_rod_cell: axis (none) -> 0 0 1; limit (none) -> lower=0 upper=0.0001 effort=1 velocity=0.0001; origin xyz=0 0 0 rpy=0 0 0 -> xyz=0.075 -0.050 0.0075 rpy=0 0 0; type fixed -> revolute
- joint object_J: parent upper_box -> base
- joint upper_body_J: axis (none) -> 0 0 1; limit (none) -> lower=0 upper=0.0001 effort=1 velocity=0.0001; origin xyz=0 0 0 rpy=0 0 0 -> xyz=0 0 0.085 rpy=0 0 0; type fixed -> revolute
- joint upper_box_J: axis (none) -> 0 0 1; limit (none) -> lower=0 upper=0.0001 effort=1 velocity=0.0001; origin xyz=0 0 0 rpy=0 0 0 -> xyz=0 0 0.015 rpy=0 0 0; type fixed -> revolute

Commit message: 추가할 건 다 했는데 rodcell에 걸리는 힘 측정이 안 됨(다음에 이어서 해보기로)

File: urdf/aidin_m1.urdf (robot description, URDF)
Before this commit: robot aidin_m1, 25 links, 24 joints
Joints:
- joint LBJ_rod_cell: axis 0 0 1 -> 1 0 0
- joint LFJ_rod_cell: axis 0 0 1 -> 1 0 0
- joint RBJ_rod_cell: axis 0 0 1 -> 1 0 0
- joint RFJ_rod_cell: axis 0 0 1 -> 1 0 0
- joint upper_body_J: axis 0 0 1 -> 1 0 0
- joint upper_box_J: axis 0 0 1 -> 1 0 0

Commit message: 에이 모르겠다

File: urdf/aidin_m1.urdf (robot description, URDF)
Before this commit: robot aidin_m1, 25 links, 24 joints
Links:
- link LB_rod_cell: mass 0.001 -> 0.1
- link LF_rod_cell: mass 0.001 -> 0.1
- link RB_rod_cell: mass 0.001 -> 0.1
- link RF_rod_cell: mass 0.001 -> 0.1
- link upper_body: mass 0.0001 -> 0.5
- link upper_box: mass 0.0001 -> 0.2
